File: Kicad/hycas.sch (KiCad schematic (older format))
At the start: 105 parts, among them J1 Conn_Coaxial, J2 S-Meter, J3 Vcc, J4 AGC Off, J5 Mute, Q1 2N3904, Q10 2N3906, Q11 2N3904, Q12 2N3904, Q2 J310, Q3 2N3904, Q4 J310, Q5 2N3904, Q6 J310, Q7 2N3906, Q8 2N3906, Q9 2N3904, T1 16T 4T FB-43-2401, U1 LM324, U2 L7809

Commit message: Add files via upload
Parts:
- Q1, Q11, Q12, Q3, Q5, Q9: symbol Transistor_BJT:2N3904_SMD -> tube:2N3904_SOT23
- Q10, Q7, Q8: symbol Transistor_BJT:2N3906_SMD -> tube:2N3906_SOT23
Connections:
- net Vin2: no longer Q7.1 (B)
Changed lines of the file:
@@
 $EndComp
 $Comp
-L Transistor_BJT:2N3904_SMD Q1
+L tube:2N3904_SOT23 Q1
 U 1 1 5CF0E0C5
 P 2300 3800
@@
 $EndComp
 $Comp
-L Transistor_BJT:2N3904_SMD Q3
+L tube:2N3904_SOT23 Q3
 U 1 1 5CF0FFD0
 P 3450 3650
@@
 $EndComp
 $Comp
-L Transistor_BJT:2N3904_SMD Q5
+L tube:2N3904_SOT23 Q5
 U 1 1 5CF10466
 P 4700 3650
@@
 	2400 2900 2400 3250
 $Comp
-L Transistor_BJT:2N3906_SMD Q7
+L tube:2N3906_SOT23 Q7
 U 1 1 5CF17517
 P 6100 3150
@@
 $EndComp
 $Comp
-L Transistor_BJT:2N3906_SMD Q8
+L tube:2N3906_SOT23 Q8
 U 1 1 5CF1A0EE
 P 7300 3150
@@
 	5600 3000 5900 3000
 Wire Wire Line
-	5900 3000 5900 3150
-Wire Wire Line
 	7500 3400 7500 3150
 $Comp
@@
 Wire Wire Line
 	7200 2950 7000 2950
-Connection ~ 7200 2950
 Wire Wire Line
 	6700 2950 6600 2950
@@
 Wire Wire Line
 	6200 2950 6200 2850
-Connection ~ 6200 2950
 Wire Wire Line
 	5900 3000 5900 2850
@@
 	-1   0    0    1
 $EndComp
-Wire Wire Line
-	5900 3550 5900 3150
-Connection ~ 5900 3150
 $Comp
 L power:GND #PWR023
@@
 $EndComp
 $Comp
-L Transistor_BJT:2N3904_SMD Q9
+L tube:2N3904_SOT23 Q9
 U 1 1 5CF47EB4
 P 7850 4400
@@
 	8750 4400 8850 4400
 $Comp
-L Transistor_BJT:2N3904_SMD Q12
+L tube:2N3904_SOT23 Q12
 U 1 1 5CF5B208
 P 9750 3800
@@
 $EndComp
 $Comp
-L Transistor_BJT:2N3904_SMD Q11
+L tube:2N3904_SOT23 Q11
 U 1 1 5CF5BEEF
 P 9000 3800
@@
 	1    0    0    -1
 $EndComp
-Wire Wire Line
-	9950 3800 10200 3800
 $Comp
 L Device:R R41
@@
 Wire Wire Line
 	10200 3800 10350 3800
-Connection ~ 10200 3800
 $Comp
 L Connector:Screw_Terminal_01x02 J5
@@
 	10650 3800 10750 3800
 $Comp
-L Transistor_BJT:2N3906_SMD Q10
+L tube:2N3906_SOT23 Q10
 U 1 1 5CF6D2D5
 P 8650 2600
@@
 Wire Wire Line
 	5050 6050 5050 6500
+Wire Wire Line
+	5900 3000 5900 3550
+Wire Wire Line
+	9950 3800 10200 3800
+Connection ~ 10200 3800
 $EndSCHEMATC

Commit message: updated version
Parts:
- R9: value 22k -> 4.7k
Changed lines of the file:
@@
 P 2650 6500
 F 0 "R9" H 2580 6454 50  0000 R CNN
-F 1 "22k" H 2580 6545 50  0000 R CNN
+F 1 "4.7k" H 2580 6545 50  0000 R CNN
 F 2 "Resistor_SMD:R_1206_3216Metric_Pad1.42x1.75mm_HandSolder" V 2580 6500 50  0001 C CNN
 F 3 "~" H 2650 6500 50  0001 C CNN
